File: SMD_Lebowski.kicad_pcb (KiCad board)
At the start: 2 copper layers, 93 parts, among them P1 Conn_01x05, P2 Conn_01x05, P3 Conn_01x05, P4 Conn_02x12_Odd_Even, P5 Conn_01x02, P6 Conn_01x03, P7 Conn_01x02, P8 Conn_01x02, Q1 BC807, Q2 BC807, Q3 BC807, Q4 BC817, U1 PIC30F4011, U2 mpc16301, U3 lm5017, U4 max809

Commit message: finished
Parts:
- P4: moved to B.Cu
- moved R11 15.9 mm to (162.3, 112.8)
- moved C11 12.5 mm to (163.7, 97.1), turned to 0 degrees
- moved C14 4.32 mm to (157.5, 87.9)
- moved R35 3.17 mm to (162.9, 85.3)
- moved C10 2.07 mm to (146.3, 127.1), turned to 270 degrees
- moved C15 1.95 mm to (165.8, 86.3), turned to 90 degrees
- moved C7 1.71 mm to (158.2, 114.6)
- moved P4 1.18 mm to (136.9, 132.8), turned to 270 degrees
- moved C2 1.03 mm to (148.3, 127.0), turned to 270 degrees
- moved C4 0.68 mm to (153.0, 123.5)
- moved R10 0.54 mm to (154.4, 127.0), turned to 270 degrees
- moved R8 0.51 mm to (150.4, 127.0), turned to 270 degrees
- moved C3 0.31 mm to (148.6, 123.5)
- moved C6 0.19 mm to (162.0, 116.3)
- moved C5 0.11 mm to (160.1, 116.3)
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Routing:
- net GND: track 0.00 -> 402.4 mm, vias 0 -> 19
- net +5V: track 0.00 -> 195.7 mm, vias 0 -> 5
- net +15V: track 0.00 -> 99.3 mm, vias 0 -> 1
- net BAT: track 0.00 -> 46.8 mm, vias 0 -> 2
- net NRES: track 0.00 -> 43.8 mm, vias 0 -> 1
- net BPOW: track 0.00 -> 42.9 mm, vias 0 -> 1
- net REV: track 0.00 -> 41.1 mm, vias 0 -> 2
- net BFB: track 0.00 -> 32.9 mm, vias 0 -> 2
- net HALL1: track 0.00 -> 32.1 mm
- net CFB: track 0.00 -> 29.7 mm, vias 0 -> 2
- net READY: track 0.00 -> 29.4 mm, vias 0 -> 1
- net AFB: track 0.00 -> 28.3 mm, vias 0 -> 2
- net Net-(C14-Pad1): track 0.00 -> 26.8 mm
- net HALL2: track 0.00 -> 25.3 mm, vias 0 -> 1
- net Net-(C10-Pad1): track 0.00 -> 23.0 mm, vias 0 -> 3
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- added copper zone on B.Cu, net GND
- added copper zone on F.Cu, net GND
Other:
- board outline added: 43 x 58.5 mm
- rule trace_min: 0.2 -> 0.01
- board text added: "Pee is stored in the balls"
